File: EagleCADs/LARC Main Board/MainBoard LARC 2017.brd (EAGLE design)
At the start: 309.9 x 198.1 mm, 31 parts, among them IC1 7805TV

Commit message: PCB Lower level finished
Parts:
- removed NEGATIVE_T1, POSITIVE_T1: (no value), adafruit:2X04
- removed R11, R12: (no value), adafruit:0207/9
- added ANALOG, JP1, JP10, JP11: (no value), pinhead:1X06
- added JP12: (no value), pinhead:1X03
- added JP2, JP3, JP4, JP5, JP6: (no value), pinhead:1X04
- added JP7, JP8, JP9: (no value), pinhead:1X02
- moved R10 324.7 mm to (214.6, 16.5)
- moved R9 324.3 mm to (214.6, 20.3)
- moved R8 324.0 mm to (214.6, 24.1)
- moved R7 323.8 mm to (214.6, 27.9)
- moved R6 323.5 mm to (214.6, 31.8)
- moved R5 323.2 mm to (214.6, 35.6)
- moved R4 322.9 mm to (214.6, 39.4)
- moved R3 322.6 mm to (214.6, 43.2)
- moved R2 322.3 mm to (214.6, 47.0)
- moved R1 322.1 mm to (214.6, 50.8)
- moved INT1 37.6 mm to (179.1, 179.1), turned to 180 degrees
- moved INT2 30.6 mm to (179.1, 174.0), turned to 180 degrees
- moved NEGATIVE_T 4.58 mm to (161.3, 188.0)
- moved POSITIVE_T 3.59 mm to (146.1, 188.0), turned to 180 degrees
- moved SWITCH_GRAL 2.54 mm to (8.89, 66.0)
Connections:
- new net A0: B1.A0, JP3.4
- new net A1: B1.A1, JP3.3
- new net A2: B1.A2, JP3.2
- new net A3: B1.A3, JP3.1
- new net A4: B1.A4, JP4.4
- new net A5: B1.A5, JP4.3
- new net A6: B1.A6, JP4.2
- new net A7: B1.A7, JP4.1
- new net ANALOGS10: ANALOG.4, B1.A10
- new net ANALOGS11: ANALOG.3, B1.A11
- new net ANALOGS12: ANALOG.2, B1.A12
- new net ANALOGS13: ANALOG.1, B1.A13
- new net ANALOGS8: ANALOG.6, B1.A8
- new net ANALOGS9: ANALOG.5, B1.A9
- new net D10: B1.10, JP12.3
- new net D11: B1.11, JP12.2
- new net D12: B1.12, JP12.1
- new net D13: B1.13
- new net D14: B1.14, JP10.1
- new net D15: B1.15, JP10.2
- new net D16: B1.16, JP10.3
- new net D17: B1.17, JP10.4
- new net D18: B1.18, JP10.5
- new net D19: B1.19, JP10.6
- new net D30: B1.30, JP1.6, R1.1
- new net D32: B1.32, JP1.5, R2.1
- new net D34: B1.34, JP1.4, R3.1
- new net D36: B1.36, JP1.3, R4.1
- new net D38: B1.38, JP1.2, R5.1
- new net D4: B1.4, JP11.6
- new net D40: B1.40, JP1.1, R6.1
- new net D42: B1.42, JP2.4, R7.1
- new net D44: B1.44, JP2.3, R8.1
- new net D46: B1.46, JP2.2, R9.1
- new net D48: B1.48, JP2.1, R10.1
- new net D5: B1.5, JP11.5
- new net D6: B1.6, JP11.4
- new net D7: B1.7, JP11.3
- new net D8: B1.8, JP11.2
- new net D9: B1.9, JP11.1
- new net GND: R1.2, R10.2, R2.2, R3.2, R4.2, R5.2, R6.2, R7.2, R8.2, R9.2
- new net SCL: B1.21, JP7.2, JP8.1, JP9.1
- new net SDA: B1.20, JP7.1, JP8.2, JP9.2
- net 5V_GRAL: now also JP6.1, JP6.2, JP6.3, JP6.4; no longer POSITIVE_T1.1, POSITIVE_T1.2, POSITIVE_T1.3, POSITIVE_T1.4, POSITIVE_T1.5, POSITIVE_T1.6, POSITIVE_T1.7, POSITIVE_T1.8
- net GND_GRAL: now also B1.GND@1, JP5.1, JP5.2, JP5.3, JP5.4; no longer NEGATIVE_T1.1, NEGATIVE_T1.2, NEGATIVE_T1.3, NEGATIVE_T1.4, NEGATIVE_T1.5, NEGATIVE_T1.6, NEGATIVE_T1.7, NEGATIVE_T1.8
Routing:
- net SCL: track 0.00 -> 312.4 mm
- net SDA: track 0.00 -> 304.8 mm
- net D40: track 0.00 -> 196.8 mm
- net D38: track 0.00 -> 193.9 mm
- net D36: track 0.00 -> 191.1 mm
- net D42: track 0.00 -> 179.2 mm
- net D34: track 0.00 -> 174.5 mm
- net D44: track 0.00 -> 173.4 mm
- net D32: track 0.00 -> 170.9 mm
- net D46: track 0.00 -> 169.4 mm
- net D48: track 0.00 -> 167.6 mm
- net D30: track 0.00 -> 167.3 mm
- net GND_GRAL: track 0.00 -> 162.6 mm, vias 0 -> 8
- net A3: track 0.00 -> 153.4 mm
- net A2: track 0.00 -> 146.5 mm
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- added copper zone on layer 16, net GND_GRAL
Other:
- board text added: "A[0..3]"
- board text added: "A[4..7]"
- board text added: "A[8..13]"
- board text added: "PULL UPS"
- board text added: "SCL"
- board text added: "SDA"
