File: EagleCADs/LARC Main Board/MainBoard LARC 2017.brd (EAGLE design)
At the start: 309.9 x 198.1 mm, 40 parts, among them IC1 7805TV

Commit message: updates to the PCB
Parts:
- moved MS_2 15.3 mm to (88.9, 35.6)
- moved JP1 11.4 mm to (237.5, 38.1)
- moved JP2 11.4 mm to (237.5, 16.5)
- moved JP3 2.54 mm to (274.3, 10.2)
Connections:
- removed net GND: R1.2, R10.2, R2.2, R3.2, R4.2, R5.2, R6.2, R7.2, R8.2, R9.2
- net GND_GRAL: now also R1.2, R10.2, R2.2, R3.2, R4.2, R5.2, R6.2, R7.2, R8.2, R9.2
Routing:
- net GND_GRAL: track 162.6 -> 139.9 mm
- net 5V_GRAL: track 480.3 -> 497.8 mm
- net 2_SHIELD1: track 94.2 -> 82.1 mm
- net D48: track 167.6 -> 156.1 mm
- net D46: track 169.4 -> 157.9 mm
- net D44: track 173.4 -> 162.0 mm
- net D42: track 179.2 -> 167.8 mm
- net D40: track 196.8 -> 185.3 mm
- net D38: track 193.9 -> 182.5 mm
- net D36: track 191.1 -> 179.6 mm
- net D34: track 174.5 -> 163.0 mm
- net D32: track 170.9 -> 159.5 mm
- net D30: track 167.3 -> 155.8 mm
- net 2_SHIELD2: track 101.0 -> 89.7 mm
- net 2_SHIELD3: track 104.1 -> 93.5 mm
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Other:
- board text added: "Roborregos 2017"

Commit message: MainBoard v1.0
Parts:
- added JP13: (no value), pinhead:1X04
- JP11: device pinhead:1X06 -> pinhead:1X04
- JP12: device pinhead:1X03 -> pinhead:1X05
- moved JP5 167.9 mm to (188.0, 5.08), turned to 0 degrees
- moved JP6 146.1 mm to (166.4, 5.08)
- moved JP11 145.3 mm to (33.0, 11.4), turned to 90 degrees
- moved JP3 45.6 mm to (229.9, 20.3), turned to 270 degrees
- moved JP9 22.9 mm to (213.4, 97.8), turned to 270 degrees
- moved JP2 18.2 mm to (229.9, 33.0)
- moved JP8 17.6 mm to (217.2, 97.8), turned to 270 degrees
- moved JP12 15.3 mm to (157.5, 85.1)
- moved JP1 12.7 mm to (229.9, 48.3)
- moved JP7 12.5 mm to (221.0, 97.8), turned to 90 degrees
- moved SWITCH_GRAL 10.2 mm to (8.89, 55.9)
- moved IC1 9.92 mm to (29.2, 67.3), turned to 90 degrees
- moved SWITCH_SERVOS 6.48 mm to (8.89, 30.5)
- moved SERVOS 6.35 mm to (21.6, 26.7), turned to 0 degrees
- moved INPUT_GRAL 5.39 mm to (21.6, 53.3), turned to 0 degrees
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Connections:
- removed net D10: B1.10, JP12.3
- removed net D11: B1.11, JP12.2
- removed net D12: B1.12, JP12.1
- removed net D9: B1.9, JP11.1
- new net PWM1_M1: B1.12, MS_1.D6
- new net PWM1_M2: B1.10, MS_2.D5
- new net PWM2_M1: B1.11, MS_1.D5
- new net PWM2_M2: B1.9, MS_2.D6
- net 5V_GRAL: now also JP11.1, JP11.2, JP11.3, JP11.4
- net 5V_SWITCH: now also R1.2, R10.2, R2.2, R3.2, R4.2, R5.2, R6.2, R7.2, R8.2, R9.2
- net D4: now also JP12.5; no longer JP11.6
- net D5: now also JP12.4; no longer JP11.5
- net D6: now also JP12.3; no longer JP11.4
- net D7: now also JP12.2; no longer JP11.3
- net D8: now also JP12.1; no longer JP11.2
- net GND_GRAL: now also JP13.1, JP13.2, JP13.3, JP13.4; no longer R1.2, R10.2, R2.2, R3.2, R4.2, R5.2, R6.2, R7.2, R8.2, R9.2
Routing:
- net 5V_SWITCH: track 267.3 -> 552.1 mm
- net PWM2_M2: track 0.00 -> 173.1 mm
- net PWM1_M2: track 0.00 -> 170.6 mm
- net PWM2_M1: track 0.00 -> 122.1 mm
- net PWM1_M1: track 0.00 -> 113.4 mm
- net 5V_GRAL: track 497.8 -> 576.1 mm
- net A0: track 129.5 -> 93.4 mm
- net A1: track 137.1 -> 106.1 mm
- net A2: track 144.0 -> 115.5 mm
- net A3: track 150.9 -> 124.9 mm
- net D30: track 155.8 -> 138.1 mm
- net GND_GRAL: track 139.9 -> 157.4 mm, vias 8 -> 7
- net D32: track 159.5 -> 142.4 mm
- net D34: track 163.0 -> 146.8 mm
- net SCL: track 312.4 -> 296.2 mm
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Other:
- board size 309.9 x 198.1 mm -> 246.4 x 198.1 mm
- board text added: "+"
- board text added: "-"
- board text removed: "A[0..3]"
- board text removed: "Derecha"
- board text removed: "Front"

Commit message: placa
Routing:
- net 1_SHIELD1: track 144.3 -> 142.5 mm
Changed lines of the file:
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@@
 <signal name="1_SHIELD1">
 <contactref element="MS_1" pad="D4"/>
-<wire x1="177.8" y1="93.98" x2="177.8" y2="118.11" width="0.6096" layer="16"/>
-<wire x1="177.8" y1="118.11" x2="179.07" y2="119.38" width="0.6096" layer="16"/>
-<wire x1="179.07" y1="119.38" x2="177.8" y2="119.38" width="0.6096" layer="16"/>
+<wire x1="180.34" y1="93.98" x2="180.34" y2="119.38" width="0.6096" layer="16"/>
+<wire x1="180.34" y1="119.38" x2="177.8" y2="119.38" width="0.6096" layer="16"/>
 <contactref element="B1" pad="28"/>
 <wire x1="186.69" y1="62.23" x2="186.69" y2="92.71" width="0.6096" layer="16"/>
-<wire x1="177.8" y1="93.98" x2="185.42" y2="93.98" width="0.6096" layer="16"/>
+<wire x1="180.34" y1="93.98" x2="185.42" y2="93.98" width="0.6096" layer="16"/>
 <wire x1="185.42" y1="93.98" x2="186.69" y2="92.71" width="0.6096" layer="16"/>
 <wire x1="110.49" y1="64.77" x2="111.76" y2="64.77" width="0.6096" layer="16"/>
